File: usb_serial.sch (KiCad schematic (older format))
At the start: 2 parts

Commit message: annotate schematic
Parts:
- gave numbers to parts that had none: 2
Changed lines of the file:
@@
 $EndDescr
 $Comp
-L thingb:HT42B534 U?
+L thingb:HT42B534 U9
 U 1 1 5C941C5F
 P 3400 2550
-F 0 "U?" H 3400 3241 39  0000 C CNN
+F 0 "U9" H 3400 3241 39  0000 C CNN
 F 1 "HT42B534" H 3400 3166 39  0000 C CNN
 F 2 "Package_SO:SOIC-16_3.9x9.9mm_P1.27mm" H 3400 2600 39  0001 C CNN
@@
 GND
 $Comp
-L Device:C_Small C?
+L Device:C_Small C14
 U 1 1 5C942CE1
 P 2300 2700
-F 0 "C?" H 2208 2654 50  0000 R CNN
+F 0 "C14" H 2208 2654 50  0000 R CNN
 F 1 "1uF" H 2208 2745 50  0000 R CNN
 F 2 "" H 2300 2700 50  0001 C CNN

Commit message: associate footprints with all parts
Parts:
- C14: footprint (none) -> Capacitor_SMD:C_0603_1608Metric_Pad1.05x0.95mm_HandSolder
Changed lines of the file:
@@
 F 0 "C14" H 2208 2654 50  0000 R CNN
 F 1 "1uF" H 2208 2745 50  0000 R CNN
-F 2 "" H 2300 2700 50  0001 C CNN
+F 2 "Capacitor_SMD:C_0603_1608Metric_Pad1.05x0.95mm_HandSolder" H 2300 2700 50  0001 C CNN
 F 3 "~" H 2300 2700 50  0001 C CNN
 	1    2300 2700
