File: thingb-eval-hw.kicad_pcb (KiCad board)
At the start: 2 copper layers, 100 x 100 mm, 70 parts, among them J1 USB_C_Receptacle_USB2.0, J2 Conn_01x06, J3 Conn_01x05, J4 SIM_Card, Q1 S9015, Q2 RU8205G, SW1 SW_Push, SW2 SW_Push, SW3 TSWB-3N-CB, U1 ESP32-WROVER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

Commit message: actually i'm ordering them today
Other:
- board text added: "rev A - 2019-04-19"
- board text removed: "rev A - 2019-04-20"
Changed lines of the file:
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@@
   (gr_line (start 117 103.5) (end 121 103.5) (layer F.SilkS) (width 0.12))
   (gr_line (start 117 86.25) (end 117 103.5) (layer F.SilkS) (width 0.12))
-  (gr_text "rev A - 2019-04-20" (at 120 103.25 90) (layer F.SilkS)
+  (gr_text "rev A - 2019-04-19" (at 120 103.25 90) (layer F.SilkS)
     (effects (font (size 1 1) (thickness 0.15)) (justify left))
   )
